Commit message: fixed assignment 1 simulation to use x-z plane and added camera 2D view

File: src/urdfs/double_pendulum.urdf (robot description, URDF)
Before this commit: robot linkage, 3 links, 2 joints
Links:
- link link B: geometry visual cylinder length=3 radius=0.05
- link link C: geometry visual cylinder length=3 radius=0.05

Commit message: update

File: src/urdfs/double_pendulum.urdf (robot description, URDF)
Before this commit: robot linkage, 3 links, 2 joints
Links:
- link link B: geometry visual cylinder length=1 radius=0.05
- link link C: geometry visual cylinder length=1 radius=0.05
Joints:
- joint joint A: limit (none) -> lower=-3.14 upper=3.14 effort=20; type continuous -> revolute
- joint joint B: limit (none) -> lower=-3.14 upper=3.14 effort=20; type continuous -> revolute

Commit message: cleanup assign 1, add assign 2.

File: src/urdfs/double_pendulum.urdf (robot description, URDF)
Before this commit: robot linkage, 3 links, 2 joints
Joints:
- joint joint A: limit (none) -> lower=-3.14 upper=3.14 effort=20; type continuous -> revolute
- joint joint B: limit (none) -> lower=-3.14 upper=3.14 effort=20; type continuous -> revolute
